Commit message: Rename ignition to gz

File: urdf/intel_realsense_d435.urdf.xacro (robot description, xacro)
@@ -153,5 +153,5 @@
         <topic>${ns}${device_namespace}/color/image_raw</topic>
         <visualize>false</visualize>
-        <ignition_frame_id>${device_namespace}_color_optical_frame</ignition_frame_id>
+        <gz_frame_id>${device_namespace}_color_optical_frame</gz_frame_id>
         <horizontal_fov>${69.0/180.0*pi}</horizontal_fov>
         <image>
@@ -170,5 +170,5 @@
         <topic>${ns}${device_namespace}/depth/image_rect_raw</topic>
         <visualize>false</visualize>
-        <ignition_frame_id>${device_namespace}_depth_optical_frame</ignition_frame_id>
+        <gz_frame_id>${device_namespace}_depth_optical_frame</gz_frame_id>
         <camera>
           <horizontal_fov>${87.0/180.0*pi}</horizontal_fov>

File: urdf/kinova.urdf.xacro (robot description, xacro)
@@ -166,5 +166,5 @@
             <optical_frame_id>${device_namespace}_color_optical_frame</optical_frame_id>
           </camera>
-          <ignition_frame_id>${device_namespace}_camera_color_frame</ignition_frame_id>
+          <gz_frame_id>${device_namespace}_camera_color_frame</gz_frame_id>
           <always_on>1</always_on>
           <update_rate>${camera_fps}</update_rate>

File: urdf/orbbec_astra.urdf.xacro (robot description, xacro)
@@ -82,5 +82,5 @@
         <topic>${ns}${device_namespace}/color/image_raw</topic>
         <visualize>false</visualize>
-        <ignition_frame_id>${ns}${device_namespace}_color_optical_frame</ignition_frame_id>
+        <gz_frame_id>${ns}${device_namespace}_color_optical_frame</gz_frame_id>
         <horizontal_fov>${60.0/180.0*pi}</horizontal_fov>
         <image>
@@ -98,5 +98,5 @@
         <topic>${ns}${device_namespace}/depth/image_raw</topic>
         <visualize>false</visualize>
-        <ignition_frame_id>${ns}${device_namespace}_depth_optical_frame</ignition_frame_id>
+        <gz_frame_id>${ns}${device_namespace}_depth_optical_frame</gz_frame_id>
         <camera>
           <horizontal_fov>${60.0/180.0*pi}</horizontal_fov>

File: urdf/ouster.urdf.xacro (robot description, xacro)
@@ -126,5 +126,5 @@
         <topic>${ns}${device_ns}ouster/points</topic>
         <frame_id>${ns}${prefix}os_lidar</frame_id>
-        <ignition_frame_id>${ns}${prefix}os_lidar</ignition_frame_id>
+        <gz_frame_id>${ns}${prefix}os_lidar</gz_frame_id>
         <always_on>true</always_on>
       </sensor>

File: urdf/slamtec_rplidar.urdf.xacro (robot description, xacro)
@@ -106,5 +106,5 @@
       <xacro:property name="dist_res" value="0.03" />
       <xacro:property name="std_dev" value="0.05" />
-      <xacro:property name="mesh" value="slamtec_rplidar_a3.dae" />
+      <xacro:property name="mesh" value="slamtec_rplidar_ax.dae" />
       <xacro:property name="collision">
         <origin xyz="0.0 0.0 ${0.041/2.0}" rpy="0.0 0.0 0.0" />
@@ -228,5 +228,5 @@
         <visualize>false</visualize>
         <topic>${ns}${device_ns}scan</topic>
-        <ignition_frame_id>${ns}${prefix}laser</ignition_frame_id>
+        <gz_frame_id>${ns}${prefix}laser</gz_frame_id>
         <ray>
           <scan>

File: urdf/stereolabs_zed.urdf.xacro (robot description, xacro)
@@ -169,5 +169,5 @@
         <topic>${ns}${device_namespace}/zed_node/rgb/image_rect_color</topic>
         <visualize>false</visualize>
-        <ignition_frame_id>${device_namespace}_center_optical_frame</ignition_frame_id>
+        <gz_frame_id>${device_namespace}_center_optical_frame</gz_frame_id>
         <camera>
           <horizontal_fov>${110.0/180.0*pi}</horizontal_fov>
@@ -188,5 +188,5 @@
         <topic>${ns}${device_namespace}/zed_node/depth</topic>
         <visualize>false</visualize>
-        <ignition_frame_id>${device_namespace}_center_optical_frame</ignition_frame_id>
+        <gz_frame_id>${device_namespace}_center_optical_frame</gz_frame_id>
         <camera>
           <horizontal_fov>${110.0/180.0*pi}</horizontal_fov>

File: urdf/teltonika_003R-00253.urdf.xacro (robot description, xacro)
@@ -54,5 +54,5 @@
         <update_rate>1</update_rate>
         <topic>${ns}${device_namespace}/fix</topic>
-        <ignition_frame_id>${ns}${device_namespace}</ignition_frame_id>
+        <gz_frame_id>${ns}${device_namespace}</gz_frame_id>
       </sensor>
     </gazebo>

File: urdf/velodyne_puck.urdf.xacro (robot description, xacro)
@@ -90,5 +90,5 @@
         <topic>${ns}${device_ns}velodyne_points</topic>
         <frame_id>${ns}${prefix}velodyne</frame_id>
-        <ignition_frame_id>${ns}${prefix}velodyne</ignition_frame_id>
+        <gz_frame_id>${ns}${prefix}velodyne</gz_frame_id>
         <always_on>true</always_on>
       </sensor>
