Commit message: Added requested receiver tf to wireless charging station (#55)
* Added requested receiver tf

Signed-off-by: Jakub Delicat <jakub.delicat@husarion.com>

* Added requested receiver tf

Signed-off-by: Jakub Delicat <jakub.delicat@husarion.com>

* Added background to tag

Signed-off-by: Jakub Delicat <jakub.delicat@husarion.com>

---------

Signed-off-by: Jakub Delicat <jakub.delicat@husarion.com>

File: urdf/wibotic_station.urdf.xacro (robot description, xacro)
@@ -18,5 +18,5 @@
   <xacro:arg name="device_namespace" default="" />
   <xacro:arg name="apriltag_image_path" default="" />
-  <xacro:arg name="apriltag_size" default="0.15" />
+  <xacro:arg name="apriltag_size" default="0.07" />
   <xacro:macro name="wibotic_station"
     params="device_namespace:=None parent_link xyz rpy">
@@ -27,5 +27,5 @@
       <xacro:property name="prefix" value="${device_namespace}_" />
     </xacro:unless>
-    <joint name="${parent_link.rstrip('_link')}_to_${prefix}wibotic_station_link_joint" type="fixed">
+    <joint name="${parent_link.rstrip('_link')}_to_${prefix}wibotic_station_joint" type="fixed">
       <origin xyz="${xyz}" rpy="${rpy}" />
       <parent link="${parent_link}" />
@@ -58,7 +58,15 @@
       </inertial>
     </link>
+    <joint name="${prefix}wibotic_station_to_${prefix}wibotic_receiver_requested_pose_joint" type="fixed">
+      <!-- This should be when docking is released for panther-docker
+      <origin xyz="0.05 0.0 0.295" rpy="0.0 0.0 ${pi}" /> -->
+      <origin xyz="${0.05 + 0.30} 0.0 0.0" rpy="0.0 0.0 ${pi}" />
+      <parent link="${prefix}wibotic_station_link" />
+      <child link="${prefix}wibotic_receiver_requested_pose_link" />
+    </joint>
+    <link name="${prefix}wibotic_receiver_requested_pose_link" />
   </xacro:macro>
   <xacro:macro name="create_apriltag"
-    params="name size:=0.2 device_namespace:=None">
+    params="name size:=$(arg apriltag_size) device_namespace:=None">
     <xacro:if value="${device_namespace == 'None'}">
       <xacro:property name="prefix" value="" />
@@ -67,5 +75,15 @@
       <xacro:property name="prefix" value="${device_namespace}_" />
     </xacro:unless>
-    <link name="${prefix}${name}_link"/>
+    <link name="${prefix}${name}_link">
+      <visual>
+        <origin xyz="0 0 0" rpy="0 0 0" />
+        <geometry>
+          <box size="${size+0.02} ${size+0.02} 0.00005" />
+        </geometry>
+        <material name="White">
+          <color rgba="1.0 1.0 1.0 1.0" />
+        </material>
+      </visual>
+      </link>
     <joint name="${name}_to_${name}_${prefix}image_link_joint" type="fixed">
       <origin xyz="0 0 0" rpy="0 -${pi/2.0} ${pi/2.0}" />
@@ -77,5 +95,5 @@
         <origin xyz="0 0 0" rpy="0 ${pi/2.0} 0" />
         <geometry>
-          <box size="${size} ${size} 0.0001" />
+          <box size="${size+0.02} ${size+0.02} 0.0001" />
         </geometry>
       </collision>
@@ -113,6 +131,6 @@
     <xacro:property name="apriltag_size_prop" value="$(arg apriltag_size)" />
     <xacro:wibotic_station
-      device_namespace="$(arg device_namespace)" parent_link="${prefix}${name}_image_link"  xyz="-0.001 0.0 ${-apriltag_size_prop/2.0 - 0.125}"
-      rpy="0 0 0 " />
+      device_namespace="$(arg device_namespace)" parent_link="${prefix}${name}_image_link"  xyz="0.21 0.0 0.115"
+      rpy="${pi} 0 0 " />
   </xacro:macro>
   <xacro:create_apriltag name="apriltag" device_namespace="$(arg device_namespace)" size="$(arg apriltag_size)" />

Commit message: requested position update (#56)
Signed-off-by: Jakub Delicat <jakub.delicat@husarion.com>

File: urdf/wibotic_station.urdf.xacro (robot description, xacro)
@@ -61,5 +61,5 @@
       <!-- This should be when docking is released for panther-docker
       <origin xyz="0.05 0.0 0.295" rpy="0.0 0.0 ${pi}" /> -->
-      <origin xyz="${0.05 + 0.30} 0.0 0.0" rpy="0.0 0.0 ${pi}" />
+      <origin xyz="${0.05 + 0.45} 0.0 0.0" rpy="0.0 0.0 ${pi}" />
       <parent link="${prefix}wibotic_station_link" />
       <child link="${prefix}wibotic_receiver_requested_pose_link" />

Commit message: Changed apriltag pose
Signed-off-by: Jakub Delicat <jakub.delicat@husarion.com>

File: urdf/wibotic_station.urdf.xacro (robot description, xacro)
@@ -58,12 +58,12 @@
       </inertial>
     </link>
-    <joint name="${prefix}wibotic_station_to_${prefix}wibotic_receiver_requested_pose_joint" type="fixed">
+    <joint name="${prefix}wibotic_station_to_${prefix}wibotic_transmitter_joint" type="fixed">
       <!-- This should be when docking is released for panther-docker
       <origin xyz="0.05 0.0 0.295" rpy="0.0 0.0 ${pi}" /> -->
-      <origin xyz="${0.05 + 0.45} 0.0 0.0" rpy="0.0 0.0 ${pi}" />
+      <origin xyz="${0.05} 0.0 0.5" rpy="0.0 0.0 ${pi}" />
       <parent link="${prefix}wibotic_station_link" />
-      <child link="${prefix}wibotic_receiver_requested_pose_link" />
+      <child link="${prefix}wibotic_transmitter_link" />
     </joint>
-    <link name="${prefix}wibotic_receiver_requested_pose_link" />
+    <link name="${prefix}wibotic_transmitter_link" />
   </xacro:macro>
   <xacro:macro name="create_apriltag"
@@ -131,5 +131,5 @@
     <xacro:property name="apriltag_size_prop" value="$(arg apriltag_size)" />
     <xacro:wibotic_station
-      device_namespace="$(arg device_namespace)" parent_link="${prefix}${name}_image_link"  xyz="0.21 0.0 0.115"
+      device_namespace="$(arg device_namespace)" parent_link="${prefix}${name}_image_link"  xyz="0.0 0.0 0.5"
       rpy="${pi} 0 0 " />
   </xacro:macro>

Commit message: Removed eval
Signed-off-by: Jakub Delicat <jakub.delicat@husarion.com>

File: urdf/wibotic_station.urdf.xacro (robot description, xacro)
@@ -61,5 +61,5 @@
       <!-- This should be when docking is released for panther-docker
       <origin xyz="0.05 0.0 0.295" rpy="0.0 0.0 ${pi}" /> -->
-      <origin xyz="${0.05} 0.0 0.5" rpy="0.0 0.0 ${pi}" />
+      <origin xyz="0.05 0.0 0.5" rpy="0.0 0.0 ${pi}" />
       <parent link="${prefix}wibotic_station_link" />
       <child link="${prefix}wibotic_transmitter_link" />

Commit message: Changed apriltag pose (#57)
* Changed apriltag pose

Signed-off-by: Jakub Delicat <jakub.delicat@husarion.com>

* Removed eval

Signed-off-by: Jakub Delicat <jakub.delicat@husarion.com>

---------

Signed-off-by: Jakub Delicat <jakub.delicat@husarion.com>

File: urdf/wibotic_station.urdf.xacro (robot description, xacro)
@@ -58,12 +58,12 @@
       </inertial>
     </link>
-    <joint name="${prefix}wibotic_station_to_${prefix}wibotic_receiver_requested_pose_joint" type="fixed">
+    <joint name="${prefix}wibotic_station_to_${prefix}wibotic_transmitter_joint" type="fixed">
       <!-- This should be when docking is released for panther-docker
       <origin xyz="0.05 0.0 0.295" rpy="0.0 0.0 ${pi}" /> -->
-      <origin xyz="${0.05 + 0.45} 0.0 0.0" rpy="0.0 0.0 ${pi}" />
+      <origin xyz="0.05 0.0 0.5" rpy="0.0 0.0 ${pi}" />
       <parent link="${prefix}wibotic_station_link" />
-      <child link="${prefix}wibotic_receiver_requested_pose_link" />
+      <child link="${prefix}wibotic_transmitter_link" />
     </joint>
-    <link name="${prefix}wibotic_receiver_requested_pose_link" />
+    <link name="${prefix}wibotic_transmitter_link" />
   </xacro:macro>
   <xacro:macro name="create_apriltag"
@@ -131,5 +131,5 @@
     <xacro:property name="apriltag_size_prop" value="$(arg apriltag_size)" />
     <xacro:wibotic_station
-      device_namespace="$(arg device_namespace)" parent_link="${prefix}${name}_image_link"  xyz="0.21 0.0 0.115"
+      device_namespace="$(arg device_namespace)" parent_link="${prefix}${name}_image_link"  xyz="0.0 0.0 0.5"
       rpy="${pi} 0 0 " />
   </xacro:macro>
